File: board-design/eagle-files/esp32-plc.brd (EAGLE design)
At the start: 100 x 80 mm, 112 parts, among them Q1 600mA/40V, Q2 600mA/40V, Q3 500mA/300V, Q4 500mA/300V, Q5 500mA/300V, Q6 500mA/300V, Q7 500mA/300V, Q8 500mA/300V

Commit message: PLC Update
Added Ethernet module.

Signed-off-by: Nicolae-Andrei Vasile <vasilenicolaeandrei@gmail.com>
Parts:
- added ETH-RJ45-C1, ETH-VDDCR-C1: 1uF, rcl:C0402
- added ETH-RJ45-R1, ETH-RJ45-R2, ETH-RJ45-R3, ETH-RJ45-R4: 49.9R, rcl:R0402
- added ETH-RJ45-R10, ETH-RJ45-R11: 10k, rcl:R0402
- added ETH-RJ45-R5, ETH-RJ45-R6: 1k, rcl:R0402
- added ETH-RJ45-R8: 12.1R (1%), rcl:R0402
- added ETH-RJ45-R9: 500R, rcl:R0402
- added ETH-VDD1A-C1, ETH-VDD2A-C1: 10uF, rcl:C0402
- added ETH-VDD1A-C2, ETH-VDD2A-C2, ETH-VDDIO-C2: 100nF, rcl:C0402
- added ETH-VDD2A-C3, ETH-VDD2A-C4, ETH-VDD2A-C5: 20pF, rcl:C0402
- added ETH-VDDCR-C2: 470pF, rcl:C0402
- added ETH-VDDIO-C1: 22uF, rcl:C/6032-28R
- added L2: (no value), SparkFun-Coils:XFL4020
- added U$105: LAN8720A-CP, my-MicrochipTechnology:QFN-24(4X4MM)
- added U$111: 7499010121A, my-WurthElektronik:RJ45-7499010121A
- added U$123: ECS-250-20-30B-AEN-TR, my-ECSInc:3.2X5MM
- moved R1-RTC 1167.9 mm to (-387.4, -1027.4)
- moved RTC-C1 1156.6 mm to (-382.3, -1022.4)
- moved EEPROM-C1 1124.1 mm to (-383.5, -1010.9)
- moved JP2 1034.1 mm to (-407.7, 139.7)
- moved JP1 1030.3 mm to (-410.2, 147.3)
- moved D6 1002.7 mm to (-410.2, 134.6)
- moved D5 998.5 mm to (-398.8, 134.6)
- moved D4 988.3 mm to (-395.0, 134.6)
- moved PSU-OUT-R4 978.3 mm to (-401.3, 129.5)
- moved F1 977.4 mm to (-411.5, 118.1)
- moved PSU-OUT-R3 973.6 mm to (-414.0, 129.5)
- moved PSU-OUT-R2 962.7 mm to (-387.4, 124.5)
- moved Q8 950.4 mm to (-403.9, 118.1)
- moved R1-RTC1 878.1 mm to (-401.3, -1022.4)
- moved C4-RTC 870.5 mm to (-391.2, -1022.4)
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Connections:
- new net ETH_NRST: ETH-RJ45-R10.1, ETH-VDD2A-C5.1, U$105.15
- new net ETH_RJ45_LED1: ETH-RJ45-R5.2, U$105.3
- new net ETH_RJ45_LED2: ETH-RJ45-R11.2, ETH-RJ45-R6.2, U$105.2
- new net ETH_RJ45_RXN: ETH-RJ45-R4.2, U$105.22, U$111.6
- new net ETH_RJ45_RXP: ETH-RJ45-R3.2, U$105.23, U$111.3
- new net ETH_RJ45_TXN: ETH-RJ45-R2.2, U$105.20, U$111.2
- new net ETH_RJ45_TXP: ETH-RJ45-R1.2, U$105.21, U$111.1
- new net ETH_VDD: ETH-RJ45-C1.1, ETH-RJ45-R1.1, ETH-RJ45-R10.2, ETH-RJ45-R2.1, ETH-RJ45-R3.1, ETH-RJ45-R4.1, ETH-VDD1A-C1.1, ETH-VDD1A-C2.1, ETH-VDD2A-C1.1, ETH-VDD2A-C2.1, ETH-VDDIO-C1.+, ETH-VDDIO-C2.1, L2.P$2, U$105.1, U$105.19, U$105.9, U$111.4, U$111.5
- new net ETH_VDDCR: ETH-VDDCR-C1.1, ETH-VDDCR-C2.1, U$105.6
- new net ETH_XTAL1: ETH-VDD2A-C3.1, U$105.5, U$123.1
- new net ETH_XTAL2: ETH-RJ45-R9.1, U$105.4
- new net N$20: ETH-RJ45-R8.2, U$105.24
- new net N$27: U$105.10
- new net N$31: U$105.11
- new net N$34: U$105.12
- new net N$35: U$105.13
- new net N$36: ETH-RJ45-R5.1, U$111.10
- new net N$37: U$105.16
- new net N$38: ETH-RJ45-R6.1, U$111.12
- new net N$39: U$105.17
- new net N$40: U$105.18
- new net N$41: U$105.7
- new net N$42: U$105.8
- new net N$43: U$105.14
- new net N$44: ETH-RJ45-R9.2, ETH-VDD2A-C4.1, U$123.3
- net 3.3V: now also L2.P$1
- net GND: now also ETH-RJ45-C1.2, ETH-RJ45-R11.1, ETH-RJ45-R8.1, ETH-VDD1A-C1.2, ETH-VDD1A-C2.2, ETH-VDD2A-C1.2, ETH-VDD2A-C2.2, ETH-VDD2A-C3.2, ETH-VDD2A-C4.2, ETH-VDD2A-C5.2, ETH-VDDCR-C1.2, ETH-VDDCR-C2.2, ETH-VDDIO-C1.-, ETH-VDDIO-C2.2, U$105.25, U$105.26, U$105.27, U$105.28, U$105.29, U$105.30, U$105.31, U$105.32, U$111.11, U$111.13, U$111.14, U$111.8, U$111.9, U$123.2, U$123.4

Commit message: PLC board design
Verifications and improvements of the hardware design.

Signed-off-by: Nicolae-Andrei Vasile <vasilenicolaeandrei@gmail.com>
Parts:
- removed C1: 1nF/1kV, rcl:C0805
- removed C4-RTC: 100pF, rcl:C0402
- removed D2: 3A/40V/500mV, SparkFun-DiscreteSemi:SMA-DIODE
- removed ETH-RJ45-R9: 500R, rcl:R0402
- removed ETH-VDDIO-C1, LTE-VBAT-C10, LTE-VBAT-C9: 22uF, rcl:C/6032-28R
- removed G1: CR2032H, battery:CR2032H
- removed JP4: (no value), pinhead:1X02
- removed R1: 42/2kV, rcl:R0805
- removed R1-RTC: 10K, rcl:R0402
- removed RS-R1: 120, rcl:R0402
- removed U$10: ESDA6V1P6, my-STMicroelectronics:SOT-666
- removed U$111: 7499010121A, my-WurthElektronik:RJ45-7499010121A
- removed U$123: ECS-250-20-30B-AEN-TR, my-ECSInc:3.2X5MM
- removed U$4: ECS-.327-12.5-12QS-TR, my-ECSInc:2X1.2
- added EEPROM_IC: M95M01-DWDW3TP/K, my-STMicroelectronics:TSSOP-8
- added ETH-C0, ETH-C3, ETH-C6: 22uF, rcl:C/6032-28R
- added ETH-C1: 1uF, rcl:C0402
- added ETH-RJ45-R12, ETH-RJ45-R7: 330, rcl:R0402
- added ETH_CRYSTAL: FL2500213Z, my-DiodesIncorporated:3.2X2.5MM
- added ETH_RJ45: 7499010121A, my-WurthElektronik:RJ45-7499010121A
- added MAX_PINH0: A, pinhead:1X01
- added MAX_PINH1: B, pinhead:1X01
- added MAX_PINH2: GND, pinhead:1X01
- added RTC-C0: 10uF, rcl:C0402
- added RTC-D0: V3PM6-M3/H, my-Vishay:DO-220AA
- added RTC-R2: 10K, rcl:R0402
- added RTC_BAT: SMTU2032-C, my-Renata:32X20MM
- added RTC_CRYSTAL: ECS-.327-7-34B-C-TR, my-ECSInc:3.2X1.5MM
- added U$101, U$102: 20, my-Vishay:MELF0204
- added U$139: GREEN, my-WurthElektronik:0603
- added U$140: RED, my-WurthElektronik:0603
- ETH-C12, ETH-C13: value 20pF -> 25pF
- ETH-C4, ETH-C7: value 10uF -> 1uF
- ETH-R2, ETH-R3, ETH-R4, ETH-R5: value 49.9R -> 49.9
- ETH-R6, ETH-R7: value 1k -> 270
- ETH-VDD2A-C5: value 20pF -> 1nF
- L2: value (none) -> TBD
- RTC-C2, RTC-C3: value 15pF -> 10pF
- RTC-C4: value 10uF -> 100pF
- U$1: value M95M01-DWMN3TP/K -> 16V; device my-STMicroelectronics:SO8 -> my-Vishay:SOT-323-3
- moved U$1 93.8 mm to (-438.1, -1087.1)
- moved RTC-C4 6.35 mm to (-391.2, -1022.4)
- renumbered EEPROM-C2 to EEPROM-C0, ETH-RJ45-C1 to ETH-C11, ETH-RJ45-R1 to ETH-R2, ETH-RJ45-R10 to ETH-R1, ETH-RJ45-R2 to ETH-R3, ETH-RJ45-R3 to ETH-R4, ETH-RJ45-R4 to ETH-R5, ETH-RJ45-R5 to ETH-R6, ETH-RJ45-R6 to ETH-R7, ETH-RJ45-R8 to ETH-R0, ETH-VDD1A-C1 to ETH-C4, ETH-VDD1A-C2 to ETH-C5, ETH-VDD2A-C1 to ETH-C7, ETH-VDD2A-C2 to ETH-C8, ETH-VDD2A-C3 to ETH-C12, ETH-VDD2A-C4 to ETH-C13, ETH-VDDCR-C1 to ETHC-9, ETH-VDDCR-C2 to ETH-C10, ETH-VDDIO-C2 to ETH-C2, R1-RTC1 to RTC-R0, U$105 to ETH_IC, U$3 to RTC_IC, U$6 to LTE_IC
Connections:
- net N$27 renamed ETH_RXER
- net N$31 renamed ETH_CRS_DV
- net N$34 renamed ETH_MDIO
- net N$35 renamed ETH_MDC
- net N$37 renamed ETH_TXEN
- net N$39 renamed ETH_TXD0
- net N$40 renamed ETH_TXD1
- net N$41 renamed ETH_RXD1
- net N$42 renamed ETH_RXD0
- net N$43 renamed ETH_NINT
- removed net N$28: JP4.2, RS-R1.2, U$11.6
- removed net N$32: JP4.1, RS-R1.1, U$11.7
- removed net N$36: ETH-R6.1, U$111.10
- removed net N$38: ETH-R7.1, U$111.12
- removed net N$44: ETH-C13.1, ETH-RJ45-R9.2, U$123.3
- removed net USIM_DATA: U$10.6
- new net LTE_PWRKEY: LTE_IC.21
- new net LTE_RESET_N: LTE_IC.20
- new net MAX_A: U$102.1, U$11.7
- new net MAX_B: U$101.1, U$11.6
- new net N$14: MAX_PINH0.1, U$1.1, U$102.2
- new net N$15: MAX_PINH1.1, U$1.2, U$101.2
- new net N$16: ETH-RJ45-R7.1, U$139.1
- new net N$17: ETH-RJ45-R12.1, U$140.1
- new net N$18: ETH-R6.2, ETH_RJ45.9
- new net N$19: ETH-R7.2, ETH_RJ45.11
- net 3.3V: now also EEPROM_IC.8, RTC-C0.1, RTC-R2.2; no longer R1-RTC.2, RTC-C4.1, U$1.8
- net ESP_VSPICLK: now also EEPROM_IC.6; no longer U$1.6
- net ESP_VSPICS0: now also EEPROM_IC.1; no longer U$1.1
- net ESP_VSPID: now also EEPROM_IC.2; no longer U$1.2
- net ESP_VSPIHD: now also EEPROM_IC.7; no longer U$1.7
- net ESP_VSPIQ: now also EEPROM_IC.5; no longer U$1.5
- net ESP_VSPIWP: now also EEPROM_IC.3; no longer U$1.3
- net ETH_RJ45_LED1: now also ETH_RJ45.10; no longer ETH-R6.2
- net ETH_RJ45_LED2: now also ETH_RJ45.12; no longer ETH-R7.2
- net ETH_RJ45_RXN: now also ETH_RJ45.6; no longer U$111.6
- net ETH_RJ45_RXP: now also ETH_RJ45.4; no longer U$111.3
- net ETH_RJ45_TXN: now also ETH_RJ45.3; no longer U$111.2
- net ETH_RJ45_TXP: now also ETH_RJ45.1; no longer U$111.1
- net ETH_VDD: now also ETH-C0.+, ETH-C1.1, ETH-C3.+, ETH-C6.+, ETH_RJ45.2, ETH_RJ45.5; no longer ETH-VDDIO-C1.+, U$111.4, U$111.5
- net ETH_XTAL1: now also ETH_CRYSTAL.1; no longer U$123.1
- net ETH_XTAL2: now also ETH-C13.1, ETH_CRYSTAL.3; no longer ETH-RJ45-R9.1
- net GND: now also EEPROM_IC.4, ETH-C0.-, ETH-C1.2, ETH-C3.-, ETH-C6.-, ETH-R6.1, ETH-R7.1, ETH-RJ45-R12.2, ETH-RJ45-R7.2, ETH_CRYSTAL.2, ETH_CRYSTAL.4, ETH_RJ45.13, ETH_RJ45.14, ETH_RJ45.8, MAX_PINH2.1, RTC-C0.2, RTC_BAT.2, U$1.3; no longer C1.1, C4-RTC.2, ETH-VDDIO-C1.-, G1.-, LTE-VBAT-C10.-, LTE-VBAT-C9.-, R1.2, U$1.4, U$10.2, U$10.5, U$111.11, U$111.13, U$111.14, U$111.8, U$111.9, U$123.2, U$123.4
- net LTE_USIM_VDD: no longer U$10.1
- net LTE_VBAT: no longer LTE-VBAT-C10.+, LTE-VBAT-C9.+
- net N$6: now also RTC-D0.2; no longer D2.C
- net N$7: now also RTC-D0.1, RTC_BAT.1; no longer D2.A, G1.+
- net P$1: no longer C1.2, R1.1
- net RS-DI: now also U$139.2
- net RS-RO: now also U$140.2
- net RTC_MFP: now also RTC-R2.1
- net RTC_VBAT: now also RTC-C4.1; no longer C4-RTC.1, R1-RTC.1
- net RTC_X1: now also RTC_CRYSTAL.1; no longer U$4.1
- net RTC_X2: now also RTC_CRYSTAL.2; no longer U$4.2
- net USIM_CLK: no longer U$10.4
- net USIM_RST: no longer U$10.3
