File: board-design/kicad-files/ESP32-PLC/RTC_EEPROM.kicad_sch (KiCad schematic)
At the start: 17 parts, among them U1 MCP7940N-xSN, U16 24LC512

Commit message: [UPDATE]
Work in progress.

Signed-off-by: Nicolae-Andrei Vasile <vasilenicolaeandrei@gmail.com>
Parts:
- gave numbers to parts that had none: 2
- renumbered C1 to C49, C70 to C50, C71 to C51, C70 to C52, C3 to C53, C3 to C54, C70 to C55, C71 to C56, D39 to D3, R9 to R60, R9 to R61, U1 to U7, U16 to U8
