File: board-design/kicad-files/ESP32-PLC/LAN8720A.kicad_sch (KiCad schematic)
At the start: 43 parts

Commit message: [UPDATE]
Finished ESP32 and ESP32-programmer board designs (few corrections to be made when manufacturer is chosen - design rules).

Signed-off-by: Nicolae-Andrei Vasile <vasilenicolaeandrei@gmail.com>
Other:
- title: PLC -> ESP32
Changed lines of the file:
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@@
   (paper "A4")
   (title_block
-    (title "PLC")
-    (date "2023-08-20")
+    (title "ESP32")
+    (date "2023-12-03")
     (rev "A")
   )

Commit message: [Final report]
Added 3D models.

Signed-off-by: Nicolae-Andrei Vasile <vasilenicolaeandrei@gmail.com>
Parts:
- gave numbers to parts that had none: 42
