File: board-design/kicad-files/SAM4E-PLC/SAM4E-PLC.kicad_sch (KiCad schematic)
At the start: 66 parts, among them J1 Conn_ARM_JTAG_SWD_10, J2 0473460001, J3 302-S101, U1 LM385M-ADJ, U2 ATSAM4E16E, Y1 ECS-160-8-33B-CTN-TR, Y2 FC-135 32.7680KA-AG0

Commit message: [UPDATE]
Work in progress.

Signed-off-by: Nicolae-Andrei Vasile <vasilenicolaeandrei@gmail.com>
Parts:
- removed J3: 302-S101, Connector_IDC:IDC-Header_2x05_P2.54mm_Vertical, symbol dk_Rectangular-Connectors-Headers-Male-Pins:302-S101
- added C43: 0.1uF/6.3V/20%/C0603, Capacitor_SMD:C_0603_1608Metric, symbol Device:C
- added C44: 10uF/16V/20%/4x5.4mm, Capacitor_SMD:CP_Elec_4x5.4, symbol Device:C_Polarized
- added D2: RB068LAM-30TFTR, Diode_SMD:D_SOD-128, symbol Device:D_Schottky
- added J3: Conn_02x05_Odd_Even, Connector_IDC:IDC-Header_2x05_P2.54mm_Vertical, symbol Connector_Generic:Conn_02x05_Odd_Even
- added J4: Conn_02x10_Odd_Even, Connector_IDC:IDC-Header_2x10_P2.54mm_Vertical, symbol Connector_Generic:Conn_02x10_Odd_Even
Connections:
- net +3V3: now also D2.2 (A)
- net CNT0: now also U2.38 (PC1); no longer U2.102 (PA0/PGMEN0)
- net CNT1: now also U2.39 (PC2); no longer U2.99 (PA1/PGMEN1)
- net ESP32_INT: now also U2.103 (PC17), J3.4 (Pin_4); no longer U2.101 (PD10)
- net GND: now also C43.2, C44.2, J3.10 (Pin_10), J3.8 (Pin_8), J4.16 (Pin_16), J4.18 (Pin_18)
- net I2C_SCL: now also J4.7 (Pin_7)
- net I2C_SDA: now also J4.9 (Pin_9)
- net IO/DI0: now also U2.47 (PD27); no longer U2.55 (PD24)
- net IO/DI3: now also U2.55 (PD24); no longer U2.47 (PD27)
- net IO/DI4: now also U2.57 (PD23); no longer U2.71 (PD28)
- net IO/DI5: now also U2.60 (PD22); no longer U2.108 (PD29)
- net IO/DI6: now also U2.63 (PD21); no longer U2.34 (PD30)
- net IO/DI7: now also U2.71 (PD28); no longer U2.2 (PD31)
- net IO/DO0: now also U2.125 (PD5); no longer U2.1 (PD0)
- net IO/DO1: now also U2.121 (PD6); no longer U2.132 (PD1)
- net IO/DO2: now also U2.119 (PD7); no longer U2.131 (PD2)
- net IO/DO3: now also U2.113 (PD8); no longer U2.128 (PD3)
- net IO/DO4: now also U2.132 (PD1); no longer U2.126 (PD4)
- net IO/DO5: now also U2.131 (PD2); no longer U2.125 (PD5)
- net IO/DO6: now also U2.128 (PD3); no longer U2.121 (PD6)
- net IO/DO7: now also U2.126 (PD4); no longer U2.119 (PD7)
- net LTE/LTE_UART_CTS: no longer U2.59 (PA25/PGMD13)
- net LTE/LTE_UART_DBG_RXD: no longer U2.75 (PA9/PGMM1)
- net LTE/LTE_UART_DBG_TXD: no longer U2.66 (PA10/PGMM2)
- net LTE/LTE_UART_DCD: no longer U2.62 (PA26/PGMD14)
- net LTE/LTE_UART_DTR: no longer U2.70 (PA27/PGMD15)
- net LTE/LTE_UART_RI: no longer U2.129 (PA29)
- net LTE/LTE_UART_RTS: no longer U2.56 (PA24/PGMD12)
- net LTE/LTE_UART_RXD: no longer U2.32 (PA21/PGMD9)
- net LTE/LTE_UART_TXD: no longer U2.37 (PA22/PGMD10)
- net LTE_AP_READY: now also U2.15 (PC30), J4.11 (Pin_11); no longer U2.92 (PD12)
- net LTE_PWRKEY: now also U2.13 (PC26), J4.15 (Pin_15); no longer U2.84 (PD14)
- net LTE_RESET_N: now also U2.12 (PC27), J4.17 (Pin_17); no longer U2.106 (PD15)
- net LTE_STATUS: now also U2.14 (PC31), J4.13 (Pin_13); no longer U2.88 (PD13)
- net SAM4E_INT: now also U2.100 (PC16), J3.6 (Pin_6); no longer U2.98 (PD11)
- net ~{RTD0_DRDY}: now also U2.110 (PD9); no longer U2.74 (PD17)
- net ~{RTD1_DRDY}: now also U2.111 (PC18); no longer U2.69 (PD18)
- net at C43.1, C43.1, C43.1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: now also C43.1, C44.1
- net at D1.1 (K): now also J3.1 (Pin_1), J3.2 (Pin_2)
- net DDM: no longer names the net of R5.2, U2.136 (PB10)
- net DDP: no longer names the net of R5.2, U2.137 (PB11)
- net RTC_MFP: no longer names the net of U2.67 (PD19)
- new net: D2.1 (K), J4.19 (Pin_19), J4.20 (Pin_20)
- new net LTE_UART_CTS: J4.4 (Pin_4), U2.59 (PA25/PGMD13)
- new net LTE_UART_DBG_RXD: J4.5 (Pin_5), U2.75 (PA9/PGMM1)
- new net LTE_UART_DBG_TXD: J4.1 (Pin_1), U2.66 (PA10/PGMM2)
- new net LTE_UART_DCD: J4.2 (Pin_2), U2.62 (PA26/PGMD14)
- new net LTE_UART_DTR: J4.3 (Pin_3), U2.70 (PA27/PGMD15)
- new net LTE_UART_RI: U2.129 (PA29)
- new net LTE_UART_RTS: U2.56 (PA24/PGMD12)
- new net LTE_UART_RXD: U2.32 (PA21/PGMD9)
- new net LTE_UART_TXD: U2.37 (PA22/PGMD10)
- no-connect marks 50 -> 81
Other:
- moved on the sheet: C47, D1, L?, U1

Commit message: [UPDATE]
Work in progress.

Signed-off-by: Nicolae-Andrei Vasile <vasilenicolaeandrei@gmail.com>
Parts:
- added JP8: SolderJumper_2_Open, Jumper:SolderJumper-2_P1.3mm_Open_Pad1.0x1.5mm, symbol Jumper:SolderJumper_2_Open
- H1, H2, H3, H4: footprint MountingHole:MountingHole_2.5mm -> MountingHole:MountingHole_2.5mm_Pad_Via
Connections:
- net ESP32_INT: now also J3.5 (Pin_5); no longer J3.4 (Pin_4)
- net Earth_Protective: now also JP8.2 (B)
- net GND: now also J3.7 (Pin_7), J3.9 (Pin_9), JP8.1 (A); no longer J3.10 (Pin_10), J3.8 (Pin_8)
- net LTE_UART_RI: now also J4.6 (Pin_6)
- net LTE_UART_RTS: now also J4.8 (Pin_8)
- net LTE_UART_RXD: now also J4.12 (Pin_12)
- net LTE_UART_TXD: now also J4.10 (Pin_10)
- net SAM4E_INT: now also J3.3 (Pin_3); no longer J3.6 (Pin_6)
- net SPI_CS0: now also J3.4 (Pin_4)
- net SPI_MISO: now also J3.6 (Pin_6)
- net SPI_MOSI: now also J3.10 (Pin_10)
- net SPI_SCK: now also J3.8 (Pin_8)
- net AI0 renamed IO/AI0
- net AI1 renamed IO/AI1
- net AI2 renamed IO/AI2
- net AI3 renamed IO/AI3
- no-connect marks 81 -> 52
Other:
- removed sheet LTE
- removed sheet RTC, EEPROM
- moved on the sheet: H1, H2, H3, H4
