File: board-design/kicad-files/SAM4E-PLC/SAM4E-PLC.kicad_sch (KiCad schematic)
At the start: 71 parts, among them J1 Conn_ARM_JTAG_SWD_10, J2 0473460001, J3 Conn_02x05_Odd_Even, J4 Conn_02x10_Odd_Even, U1 LM385M-ADJ, U2 ATSAM4E16E, Y1 ECS-160-8-33B-CTN-TR, Y2 FC-135 32.7680KA-AG0

Commit message: [UPDATE]
Completed SAM4E-PLC board design.

Signed-off-by: Nicolae-Andrei Vasile <vasilenicolaeandrei@gmail.com>
Connections:
- net Earth_Protective: now also J2.SH, RV1.2, RV2.2
Other:
- note added: "Connections"
- title: (none) -> SAM4E
- moved on the sheet: D1, D2, J3, J4, JP8

Commit message: [Final report]
Added 3D models.

Signed-off-by: Nicolae-Andrei Vasile <vasilenicolaeandrei@gmail.com>
Parts:
- gave numbers to parts that had none: 1
- renumbered C47 to C1, C44 to C10, C3 to C11, C3 to C12, C3 to C13, C43 to C14, C44 to C15, C3 to C16, C43 to C17, C44 to C18, C43 to C19, C44 to C2, C44 to C20, C43 to C21, C44 to C22, C43 to C23, C44 to C24, C43 to C25, C43 to C26, C43 to C27, C43 to C28, C43 to C29, C43 to C3, C43 to C30, C43 to C31, C43 to C32, C48 to C33, C49 to C34, C3 to C35, C3 to C36, C5 to C4, C44 to C5, C5 to C6, C43 to C7, C3 to C8, C3 to C9, JP8 to JP3, R49 to R1, R40 to R10, R40 to R11, R40 to R12, R40 to R13, R49 to R2, R49 to R3, R49 to R4, R40 to R5, R5 to R6, R5 to R7, R5 to R8, R40 to R9
