File: board-design/kicad-files/SAM4E-PLC/SAM4E-PLC.kicad_pcb (KiCad board)
At the start: 2 copper layers, 86.1 x 174.1 mm, 351 parts, among them J1 Conn_ARM_JTAG_SWD_10, J2 0473460001, J3 302-S101, J4 SF53S006VCBR2000, J5 Screw_Terminal_01x11, J6 Screw_Terminal_01x11, J7 Screw_Terminal_01x11, J8 Screw_Terminal_01x11, Q1 BC817, Q10 BC807, Q11 BC807, Q12 BC807, Q13 BC817, Q2 BC817, Q3 BC807, Q4 BC807, Q5 BC807, Q6 BC807, Q7 BC807, Q8 BC807, Q9 BC807, U1 LM385M-ADJ, U10 MAX31865xAP, U11 ULN2803CDWR, U12 74AC14SCX, U13 SN74HC240DBR, U14 LM2576HVS-3.3, U15 MCP7940N-xSN, U2 ATSAM4E16E, U3 EC21, U4 TXS0108EPW, U5 TXS0108EPW, U6 SN65HVD234, U7 SN65HVD230DR, U7 SN65HVD234, U8 MAX31865xAP, U9 MAX3485ESA+T, Y1 ECS-160-8-33B-CTN-TR, Y2 FC-135 32.7680KA-AG0

Commit message: [IN PROGRESS]
SAM4E-PLC PCB design in progress.

Signed-off-by: Nicolae-Andrei Vasile <vasilenicolaeandrei@gmail.com>
Parts:
- removed the U7 at (474.7, 11.8)
- added C10: 12pF/6.3V/10%/C0603, Capacitor_SMD:C_0603_1608Metric, F.Cu at (320.4, 30.0)
- added C11: 12pF/6.3V/10%/C0603, Capacitor_SMD:C_0603_1608Metric, F.Cu at (320.4, 32.5)
- added C32: 12pF/6.3V/10%/C0603, Capacitor_SMD:C_0603_1608Metric, F.Cu at (320.4, 35.0)
- added C33: 12pF/6.3V/10%/C0603, Capacitor_SMD:C_0603_1608Metric, F.Cu at (320.4, 37.5)
- added C84: 1uF/16V/20%/4x5.4mm, Capacitor_SMD:CP_Elec_4x5.4, F.Cu at (139.1, 134.6)
- added C85: 1uF/16V/20%/4x5.4mm, Capacitor_SMD:CP_Elec_4x5.4, F.Cu at (139.1, 142.2)
- added C86: 1uF/16V/20%/4x5.4mm, Capacitor_SMD:CP_Elec_4x5.4, F.Cu at (139.1, 149.9)
- added C87: 1uF/16V/20%/4x5.4mm, Capacitor_SMD:CP_Elec_4x5.4, F.Cu at (139.1, 157.5)
- added C93: 22uF/6.3V/20%/C0603, Capacitor_SMD:C_0603_1608Metric, F.Cu at (-94.8, 26.0)
- moved C1 421.1 mm to (348.1, 22.9)
- moved C12 421.1 mm to (348.1, 35.5)
- moved C13 421.1 mm to (334.4, 23.6)
- moved C14 421.1 mm to (348.1, 38.0)
- moved C15 421.1 mm to (348.1, 40.5)
- moved C16 421.1 mm to (342.2, 0.24)
- moved C17 421.1 mm to (348.1, 43.0)
- moved C18 421.1 mm to (342.2, 6.09)
- moved C19 421.1 mm to (352.1, 22.9)
- moved C2 421.1 mm to (334.4, 0.24)
- moved C20 421.1 mm to (342.2, 11.9)
- moved C21 421.1 mm to (352.1, 25.4)
- moved C22 421.1 mm to (342.2, 17.8)
- moved C23 421.1 mm to (352.1, 27.9)
- moved C24 421.1 mm to (352.1, 30.4)
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- renumbered C80 to C79, C81 to C80, C79 to C81, D34 to D32, D35 to D33, D36 to D34, D37 to D35, D38 to D36, D32 to D37, D33 to D38, R99 to R100, R100 to R101, R101 to R102, R102 to R103, R115 to R107, R116 to R108, R117 to R109, R118 to R110, R107 to R111, R108 to R112, R109 to R113, R110 to R114, R111 to R115, R112 to R116, R113 to R117, R114 to R118, R103 to R99
Connections:
- R104 pad 2: /IO/DO1 -> Net-(JP16-C)
- R105 pad 2: /IO/DO2 -> Net-(JP13-C)
- R106 pad 2: /IO/DO3 -> Net-(JP17-C)
- R107 pad 2: /IO/DO7 -> Net-(JP18-C)
- R108 pad 2: /IO/DO6 -> Net-(JP14-C)
- R109 pad 2: /IO/DO5 -> Net-(JP19-C)
- R110 pad 2: /IO/DO4 -> Net-(JP15-C)
- R99 pad 2: /IO/DO0 -> Net-(JP12-C)
Routing:
- net +3V3: track 24.9 -> 72.2 mm
- net Net-(U8-DVDD): track 0.00 -> 33.8 mm
- net Net-(U10-DVDD): track 0.00 -> 33.7 mm
- net Net-(JP15-C): track 0.00 -> 19.4 mm
- net Net-(JP12-C): track 0.00 -> 19.4 mm
- net MCV_RTD1_RTDIN-: track 0.00 -> 17.5 mm
- net Net-(D38-K): track 0.00 -> 17.3 mm
- net MCV_RTD0_RTDIN-: track 0.00 -> 16.4 mm
- net Net-(JP19-C): track 0.00 -> 15.6 mm
- net Net-(JP16-C): track 0.00 -> 15.6 mm
- net Net-(U11-8C): track 0.00 -> 15.2 mm
- net Net-(U11-1C): track 0.00 -> 15.2 mm
- net Net-(D37-K): track 0.00 -> 14.9 mm
- net Net-(U11-2C): track 0.00 -> 12.7 mm
- net Net-(U11-7C): track 0.00 -> 12.7 mm
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
Commit message: [UPDATE]
Work in progress.

Signed-off-by: Nicolae-Andrei Vasile <vasilenicolaeandrei@gmail.com>
Parts:
- removed the D32 at (121.9, 72.4)
- removed the D33 at (121.9, 67.3)
- removed the D34 at (121.9, 62.2)
- removed the D35 at (121.9, 57.1)
- removed the D36 at (121.9, 36.8)
- removed D39, D40, D41: LED, LED_SMD:LED_0805_2012Metric
- removed the R104 at (121.9, 69.2)
- removed the R105 at (121.9, 64.1)
- removed the R106 at (121.9, 59.1)
- removed the R107 at (121.9, 38.7)
- removed the R108 at (121.9, 43.8)
- removed the R109 at (121.9, 48.9)
- removed the R110 at (121.9, 54.0)
- removed the R99 at (121.9, 74.3)
- added D1: RB068LAM-30TFTR, Diode_SMD:D_SOD-128, F.Cu at (377.8, 27.9)
- added D38: 20V/0.5A/0.5V (NSR0620P2T5G), Diode_SMD:D_SOD-923, F.Cu at (-158.1, 156.8)
- added H1: MountingHole, MountingHole:MountingHole_2.5mm, F.Cu at (94.2, 25.1)
- added H2: MountingHole, MountingHole:MountingHole_2.5mm, F.Cu at (144.2, 25.1)
- added H3: MountingHole, MountingHole:MountingHole_2.5mm, F.Cu at (144.2, 187.1)
- added H4: MountingHole, MountingHole:MountingHole_2.5mm, F.Cu at (94.2, 187.1)
- added JP1: SolderJumper_3_Open, Jumper:SolderJumper-3_P1.3mm_Open_Pad1.0x1.5mm, F.Cu at (440.7, 17.8)
- added JP2: SolderJumper_3_Open, Jumper:SolderJumper-3_P1.3mm_Open_Pad1.0x1.5mm, F.Cu at (440.7, 21.6)
- added U16: 24LC512, Package_SO:SOIC-8_3.9x4.9mm_P1.27mm, F.Cu at (-142.2, 161.9)
- BT1: value CR2032 (Keystone 1057) -> CR2032 (Panasonic vertical); footprint Battery:BatteryHolder_Keystone_1057_1x2032 -> Battery:Battery_Panasonic_CR2032-VS1N_Vertical_CircularHoles
- D35: renamed from D42; value RB075BM40SFHHTL -> RB088LAM-40TFTR; footprint digikey-footprints:TO-252-3 -> Diode_SMD:D_SOD-128
- moved D37 398.2 mm to (275.6, -50.8), turned to 180 degrees
- moved R114 375.1 mm to (282.6, -50.8), turned to 90 degrees
- moved R113 370.2 mm to (279.4, -48.3)
- moved Q13 366.5 mm to (279.4, -50.8), turned to 180 degrees
- moved R112 365.7 mm to (275.6, -48.3), turned to 180 degrees
- moved J1 294.1 mm to (88.9, 76.8)
- moved RV1 288.1 mm to (82.7, 108.6), turned to 90 degrees
- moved R4 287.6 mm to (95.2, 87.0)
- moved RV2 285.5 mm to (84.7, 108.6), turned to 90 degrees
- moved R10 284.7 mm to (88.5, 108.6), turned to -90 degrees
- moved R6 279.2 mm to (86.6, 108.6), turned to 90 degrees
- moved R7 277.7 mm to (88.5, 112.4)
- moved R8 277.5 mm to (88.5, 114.3)
- moved C7 276.6 mm to (83.5, 111.1)
- moved J2 268.5 mm to (78.1, 113.7), turned to 90 degrees
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- renumbered C81 to C79, C79 to C80, C80 to C81, D9 to D10, D10 to D11, D11 to D12, D12 to D13, D13 to D14, D14 to D15, D15 to D16, D16 to D17, D17 to D18, D18 to D19, D1 to D2, D19 to D20, D20 to D21, D21 to D22, D22 to D23, D23 to D24, D24 to D25, D25 to D26, D26 to D27, D27 to D28, D28 to D29, D2 to D3, D29 to D30, D30 to D31, D31 to D32, D37 to D33, D38 to D34, D43 to D36, D44 to D37, D3 to D4, D4 to D5, D5 to D6, D6 to D7, D7 to D8, D8 to D9, JP17 to JP12, JP16 to JP13, JP19 to JP14, JP18 to JP15, JP13 to JP16, JP12 to JP17, JP15 to JP18, JP14 to JP19, R101 to R100, R102 to R101, R103 to R102, R111 to R103, R112 to R104, R113 to R105, R114 to R106, R115 to R107, R116 to R108, R117 to R109, R118 to R110, R119 to R111, R120 to R112, R121 to R113, R122 to R114, R123 to R115, R124 to R116, R100 to R99
Connections:
- F1 pad 2: /IO/MCV_DO0 -> /IO/MCV_DO3
- F13 pad 2: Net-(D42-A) -> Net-(D35-A)
- F2 pad 2: /IO/MCV_DO1 -> /IO/MCV_DO2
- F3 pad 2: /IO/MCV_DO2 -> /IO/MCV_DO1
- F4 pad 2: /IO/MCV_DO3 -> /IO/MCV_DO0
- F5 pad 2: /IO/MCV_DO4 -> /IO/MCV_DO7
- F6 pad 2: /IO/MCV_DO5 -> /IO/MCV_DO6
- F7 pad 2: /IO/MCV_DO6 -> /IO/MCV_DO5
- F8 pad 2: /IO/MCV_DO7 -> /IO/MCV_DO4
- J3 pad 2: +3V3 -> Net-(D1-K)
- J5 pad 10: /IO/MCV_DO6 -> /IO/MCV_DO5
- J5 pad 11: /IO/MCV_DO7 -> /IO/MCV_DO4
- J5 pad 4: /IO/MCV_DO0 -> /IO/MCV_DO3
- J5 pad 7: /IO/MCV_DO3 -> /IO/MCV_DO0
- J5 pad 8: /IO/MCV_DO4 -> /IO/MCV_DO7
- J5 pad 9: /IO/MCV_DO5 -> /IO/MCV_DO6
- J7 pad 10: MCV_RTD1_RTDIN- -> MCV_RTD1_RTDIN+
- J7 pad 11: MCV_RTD1_FORCE- -> MCV_RTD1_FORCE+
- J7 pad 4: MCV_RTD0_FORCE+ -> MCV_RTD0_FORCE-
- J7 pad 5: MCV_RTD0_RTDIN+ -> MCV_RTD0_RTDIN-
- J7 pad 6: MCV_RTD0_RTDIN- -> MCV_RTD0_RTDIN+
- J7 pad 7: MCV_RTD0_FORCE- -> MCV_RTD0_FORCE+
- J7 pad 8: MCV_RTD1_FORCE+ -> MCV_RTD1_FORCE-
- J7 pad 9: MCV_RTD1_RTDIN+ -> MCV_RTD1_RTDIN-
- JP12 pad 2: Net-(JP17-C) -> Net-(JP12-C)
- JP13 pad 2: Net-(JP16-C) -> Net-(JP13-C)
- JP14 pad 2: Net-(JP19-C) -> Net-(JP14-C)
- JP15 pad 2: Net-(JP18-C) -> Net-(JP15-C)
- JP16 pad 2: Net-(JP13-C) -> Net-(JP16-C)
- JP17 pad 2: Net-(JP12-C) -> Net-(JP17-C)
- JP18 pad 2: Net-(JP15-C) -> Net-(JP18-C)
- JP19 pad 2: Net-(JP14-C) -> Net-(JP19-C)
Routing:
- net VIN_24V: track 0.00 -> 171.7 mm
- net /IO/DO0: track 0.00 -> 125.4 mm, vias 0 -> 1
- net /IO/DO7: track 0.00 -> 122.1 mm, vias 0 -> 1
- net /IO/DO6: track 0.00 -> 108.7 mm, vias 0 -> 1
- net /IO/DO1: track 0.00 -> 107.9 mm, vias 0 -> 1
- net /IO/DO5: track 0.00 -> 95.4 mm, vias 0 -> 1
- net /IO/DO2: track 0.00 -> 93.6 mm, vias 0 -> 1
- net /IO/DO4: track 0.00 -> 82.0 mm, vias 0 -> 1
- net /IO/DO3: track 0.00 -> 77.0 mm, vias 0 -> 1
- net +24V: track 7.25 -> 80.0 mm
- net /IO/DI0: track 3.90 -> 65.3 mm, vias 0 -> 1
- net Net-(JP15-C): track 19.4 -> 73.2 mm, vias 0 -> 2
- net Net-(JP19-C): track 15.6 -> 69.1 mm, vias 0 -> 2
- net /IO/DI1: track 3.90 -> 57.1 mm, vias 0 -> 1
- net Net-(JP14-C): track 11.8 -> 64.0 mm, vias 0 -> 2
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
Commit message: [UPDATE]
Work in progress.

Signed-off-by: Nicolae-Andrei Vasile <vasilenicolaeandrei@gmail.com>
Parts:
- added C30: 0.1uF/6.3V/20%/C0603, Capacitor_SMD:C_0603_1608Metric, F.Cu at (125.1, 121.3)
- moved JP1 335.4 mm to (125.1, 131.4), turned to 180 degrees
- moved JP2 329.3 mm to (130.2, 131.4), turned to 180 degrees
- moved U1 280.5 mm to (123.8, 141.0), turned to 90 degrees
- moved C31 278.6 mm to (88.9, 116.8), turned to 180 degrees
- moved C3 276.7 mm to (102.2, 125.7), turned to 180 degrees
- moved L2 276.2 mm to (91.4, 119.4), turned to 180 degrees
- moved C24 273.6 mm to (102.2, 121.9)
- moved R13 273.3 mm to (89.4, 121.9), turned to 180 degrees
- moved C28 271.9 mm to (106.0, 90.8), turned to 90 degrees
- moved C19 271.9 mm to (120.0, 87.6), turned to 90 degrees
- moved C32 271.9 mm to (91.4, 125.7)
- moved C5 271.7 mm to (106.7, 126.4), turned to -90 degrees
- moved C27 270.6 mm to (118.1, 87.6), turned to 90 degrees
- moved C12 270.4 mm to (120.7, 126.4), turned to -90 degrees
- moved C20 270.3 mm to (111.1, 85.7)
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- renumbered C99 to C100, C100 to C101, C101 to C102, C102 to C103, C30 to C31, C31 to C32, C32 to C33, C33 to C34, C34 to C35, C35 to C36, C36 to C37, C37 to C38, C38 to C39, C39 to C40, C40 to C41, C41 to C42, C42 to C43, C43 to C44, C44 to C45, C45 to C46, C46 to C47, C47 to C48, C48 to C49, C49 to C50, C50 to C51, C51 to C52, C52 to C53, C53 to C54, C54 to C55, C55 to C56, C56 to C57, C57 to C58, C58 to C59, C59 to C60, C60 to C61, C61 to C62, C62 to C63, C63 to C64, C64 to C65, C65 to C66, C66 to C67, C67 to C68, C68 to C69, C69 to C70, C70 to C71, C71 to C72, C72 to C73, C73 to C74, C74 to C75, C75 to C76, C76 to C77, C77 to C78, C78 to C79, C79 to C80, C80 to C81, C81 to C82, C82 to C83, C83 to C84, C84 to C85, C85 to C86, C86 to C87, C87 to C88, C88 to C89, C89 to C90, C90 to C91, C91 to C92, C92 to C93, C93 to C94, C94 to C95, C95 to C96, C96 to C97, C97 to C98, C98 to C99
Connections:
- C85 pad 1: /AI0 -> /AI3
- C86 pad 1: /AI1 -> /AI2
- C87 pad 1: /AI2 -> /AI1
- C88 pad 1: /AI3 -> /AI0
- F10 pad 1: /IO/MCV_AI1 -> /IO/MCV_AI2
- F11 pad 1: /IO/MCV_AI2 -> /IO/MCV_AI1
- F12 pad 1: /IO/MCV_AI3 -> /IO/MCV_AI0
- F9 pad 1: /IO/MCV_AI0 -> /IO/MCV_AI3
- J8 pad 4: /IO/MCV_AI0 -> /IO/MCV_AI3
- J8 pad 5: /IO/MCV_AI1 -> /IO/MCV_AI2
- J8 pad 6: /IO/MCV_AI2 -> /IO/MCV_AI1
- J8 pad 7: /IO/MCV_AI3 -> /IO/MCV_AI0
- R107 pad 2: /AI0 -> /AI3
- R108 pad 2: /AI1 -> /AI2
- R109 pad 2: /AI2 -> /AI1
- R110 pad 2: /AI3 -> /AI0
Routing:
- net /RS_RO: track 0.00 -> 98.6 mm
- net +3V3: track 100.8 -> 198.6 mm
- net /RS_DI: track 0.00 -> 94.9 mm
- net /AI0: track 7.41 -> 73.8 mm, vias 1 -> 0
- net /AI1: track 7.41 -> 65.7 mm, vias 1 -> 0
- net /AI2: track 7.41 -> 57.2 mm, vias 1 -> 0
- net Net-(U2-VDDOUT): track 0.00 -> 48.9 mm
- net /AI3: track 7.41 -> 48.9 mm, vias 1 -> 0
- net Net-(U2-VDDIN): track 0.00 -> 41.1 mm
- net Net-(U1-K): track 0.00 -> 35.2 mm
- net Net-(JP2-C): track 0.00 -> 24.8 mm
- net Net-(U2-VDDPLL): track 0.00 -> 23.9 mm
- net Net-(JP1-C): track 0.00 -> 23.1 mm
- net Net-(D34-K): track 24.1 -> 7.98 mm
- net /DDP: track 6.04 -> 17.4 mm
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
Commit message: [UPDATE]
Work in progress.

Signed-off-by: Nicolae-Andrei Vasile <vasilenicolaeandrei@gmail.com>
Parts:
- added C2: 10uF/16V/20%/4x5.4mm, Capacitor_SMD:CP_Elec_4x5.4, F.Cu at (98.4, 125.1)
- added C3: 0.1uF/6.3V/20%/C0603, Capacitor_SMD:C_0603_1608Metric, F.Cu at (102.9, 124.5)
- added D2: RB068LAM-30TFTR, Diode_SMD:D_SOD-128, F.Cu at (110.5, 172.1)
- added J4: Conn_02x10_Odd_Even, Connector_IDC:IDC-Header_2x10_P2.54mm_Vertical, F.Cu at (116.1, 150.5)
- J3: value 302-S101 -> Conn_02x05_Odd_Even
- moved R9 303.2 mm to (87.0, 97.2), turned to -90 degrees
- moved S1 283.8 mm to (84.2, 93.9), turned to -90 degrees
- moved D1 281.3 mm to (135.9, 171.4), turned to -90 degrees
- moved R11 276.5 mm to (124.5, 148.4), turned to 90 degrees
- moved J3 274.9 mm to (130.3, 167.0), turned to 180 degrees
- moved R12 274.5 mm to (126.4, 149.2), turned to -90 degrees
- moved C16 265.3 mm to (116.8, 90.2), turned to 90 degrees
- moved C1 259.5 mm to (95.2, 81.3), turned to 180 degrees
- moved L1 257.1 mm to (102.2, 121.3)
- moved JP3 36.1 mm to (100.3, 186.1), turned to 180 degrees
- moved R51 34.4 mm to (100.3, 183.6), turned to 0 degrees
- moved R47 33.3 mm to (100.3, 181.0), turned to 0 degrees
- moved R42 32.1 mm to (104.1, 188.6), turned to 180 degrees
- moved R41 25.8 mm to (104.1, 181.0), turned to 180 degrees
- moved R39 24.9 mm to (109.2, 188.6), turned to 0 degrees
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- renumbered C8 to C10, C98 to C100, C99 to C101, C100 to C102, C101 to C103, C102 to C104, C103 to C105, C9 to C11, C10 to C12, C11 to C13, C12 to C14, C13 to C15, C14 to C16, C15 to C17, C16 to C18, C17 to C19, C18 to C20, C19 to C21, C20 to C22, C21 to C23, C22 to C24, C23 to C25, C24 to C26, C25 to C27, C26 to C28, C27 to C29, C28 to C30, C29 to C31, C30 to C32, C31 to C33, C32 to C34, C33 to C35, C34 to C36, C35 to C37, C36 to C38, C37 to C39, C2 to C4, C38 to C40, C39 to C41, C40 to C42, C41 to C43, C42 to C44, C43 to C45, C44 to C46, C45 to C47, C46 to C48, C47 to C49, C3 to C5, C48 to C50, C49 to C51, C50 to C52, C51 to C53, C52 to C54, C53 to C55, C54 to C56, C55 to C57, C56 to C58, C57 to C59, C4 to C6, C58 to C60, C59 to C61, C60 to C62, C61 to C63, C62 to C64, C63 to C65, C64 to C66, C65 to C67, C66 to C68, C67 to C69, C5 to C7, C68 to C70, C69 to C71, C70 to C72, C71 to C73, C72 to C74, C73 to C75, C74 to C76, C75 to C77, C76 to C78, C77 to C79, C6 to C8, C78 to C80, C79 to C81, C80 to C82, C81 to C83, C82 to C84, C83 to C85, C84 to C86, C85 to C87, C86 to C88, C87 to C89, C7 to C9, C88 to C90, C89 to C91, C90 to C92, C91 to C93, C92 to C94, C93 to C95, C94 to C96, C95 to C97, C96 to C98, C97 to C99, D9 to D10, D10 to D11, D11 to D12, D12 to D13, D13 to D14, D14 to D15, D15 to D16, D16 to D17, D17 to D18, D18 to D19, D19 to D20, D20 to D21, D21 to D22, D22 to D23, D23 to D24, D24 to D25, D25 to D26, D26 to D27, D27 to D28, D28 to D29, D2 to D3, D29 to D31, D31 to D33, D33 to D35, D35 to D36, D36 to D37, D37 to D38, D38 to D39, D3 to D4, D4 to D5, D5 to D6, D6 to D7, D7 to D8, D8 to D9, J4 to J5, J5 to J6, J6 to J7, J7 to J8, J8 to J9, Q12 to Q11, Q11 to Q12, R102 to R100, R99 to R101, R100 to R102, R96 to R95, R95 to R96, R98 to R97, R97 to R98, R101 to R99
Connections:
- net /DDM renamed Net-(U2-PB10)
- net /DDP renamed Net-(U2-PB11)
- D35 pad 1: Net-(D33-K) (its old number) -> Net-(D35-K)
- J3 pad 1: /SPI_MOSI -> Net-(D1-K)
- J3 pad 3: Earth_Protective -> unconnected-(J3-Pin_3-Pad3)
- J3 pad 5: /SPI_CS0 -> unconnected-(J3-Pin_5-Pad5)
- J3 pad 7: /SPI_SCK -> unconnected-(J3-Pin_7-Pad7)
- J3 pad 9: /SPI_MISO -> unconnected-(J3-Pin_9-Pad9)
- J9 pad 10: MCV_CAN1_H -> MCV_CAN0_H
- J9 pad 11: MCV_CAN1_L -> MCV_CAN0_L
- J9 pad 8: MCV_CAN0_H -> MCV_CAN1_H
- J9 pad 9: MCV_CAN0_L -> MCV_CAN1_L
- JP3 pad 2: MCV_CAN0_H -> MCV_CAN1_H
- JP4 pad 2: MCV_CAN1_H -> MCV_CAN0_H
- R101 pad 2: Net-(D33-K) (its old number) -> Net-(D35-K)
- R102 pad 1: Net-(D33-K) (its old number) -> Net-(D35-K)
- R115 pad 2: /RTC_MFP -> /RTC, EEPROM/RTC_MFP
- R14 pad 1: /LTE_PWRKEY -> /LTE/LTE_PWRKEY
- R15 pad 1: /LTE_RESET_N -> /LTE/LTE_RESET_N
- R34 pad 2: /LTE_AP_READY -> /LTE/LTE_AP_READY
- R36 pad 1: /LTE_STATUS -> /LTE/LTE_STATUS
- R39 pad 1: /CAN0_RS -> /CAN1_RS
- R40 pad 1: /CAN0_D -> /CAN1_D
- R41 pad 1: /CAN0_EN -> /CAN1_EN
- R42 pad 1: /CAN0_R -> /CAN1_R
- R43 pad 1: /CAN1_RS -> /CAN0_RS
- R44 pad 1: /CAN1_D -> /CAN0_D
- R45 pad 1: /CAN1_EN -> /CAN0_EN
- R46 pad 1: /CAN1_R -> /CAN0_R
- R51 pad 1: MCV_CAN0_L -> MCV_CAN1_L
- R52 pad 1: MCV_CAN1_L -> MCV_CAN0_L
- U10 pad 16: /SPI_CS2 -> /SPI_CS1
- U12 pad 1: Net-(D33-K) (its old number) -> Net-(D34-K)
- U12 pad 3: Net-(D34-K) -> Net-(D35-K)
- U15 pad 5: /I2C_SCL -> /RTC, EEPROM/SDA
- U15 pad 6: /I2C_SDA -> /RTC, EEPROM/SCL
- U15 pad 7: /RTC_MFP -> /RTC, EEPROM/RTC_MFP
- U16 pad 5: /I2C_SCL -> /RTC, EEPROM/SDA
- U16 pad 6: /I2C_SDA -> /RTC, EEPROM/SCL
- U2 pad 1: /IO/DO0 -> unconnected-(U2-PD0-Pad1)
- U2 pad 100: unconnected-(U2-PC16-Pad100) -> /SAM4E_INT
- U2 pad 101: /ESP32_INT -> unconnected-(U2-PD10-Pad101)
- U2 pad 102: /CNT0 -> unconnected-(U2-PA0/PGMEN0-Pad102)
- U2 pad 103: unconnected-(U2-PC17-Pad103) -> /ESP32_INT
- U2 pad 106: /LTE_RESET_N -> unconnected-(U2-PD15-Pad106)
- U2 pad 108: /IO/DI5 -> unconnected-(U2-PD29-Pad108)
- U2 pad 110: unconnected-(U2-PD9-Pad110) -> /~{RTD0_DRDY}
- U2 pad 111: unconnected-(U2-PC18-Pad111) -> /~{RTD1_DRDY}
- U2 pad 113: unconnected-(U2-PD8-Pad113) -> /IO/DO3
- U2 pad 119: /IO/DO7 -> /IO/DO2
- U2 pad 12: unconnected-(U2-PC27-Pad12) -> /LTE_RESET_N
- U2 pad 121: /IO/DO6 -> /IO/DO1
- U2 pad 125: /IO/DO5 -> /IO/DO0
- U2 pad 126: /IO/DO4 -> /IO/DO7
- U2 pad 128: /IO/DO3 -> /IO/DO6
- U2 pad 129: /LTE/LTE_UART_RI -> /LTE_UART_RI
- U2 pad 13: unconnected-(U2-PC26-Pad13) -> /LTE_PWRKEY
- U2 pad 131: /IO/DO2 -> /IO/DO5
- U2 pad 132: /IO/DO1 -> /IO/DO4
- U2 pad 14: unconnected-(U2-PC31-Pad14) -> /LTE_STATUS
- U2 pad 15: unconnected-(U2-PC30-Pad15) -> /LTE_AP_READY
- U2 pad 2: /IO/DI7 -> unconnected-(U2-PD31-Pad2)
- U2 pad 32: /LTE/LTE_UART_RXD -> /LTE_UART_RXD
- U2 pad 34: /IO/DI6 -> unconnected-(U2-PD30-Pad34)
- U2 pad 37: /LTE/LTE_UART_TXD -> /LTE_UART_TXD
- U2 pad 38: unconnected-(U2-PC1-Pad38) -> /CNT0
- U2 pad 39: unconnected-(U2-PC2-Pad39) -> /CNT1
- U2 pad 47: /IO/DI3 -> /IO/DI0
- U2 pad 55: /IO/DI0 -> /IO/DI3
- U2 pad 56: /LTE/LTE_UART_RTS -> /LTE_UART_RTS
- U2 pad 57: unconnected-(U2-PD23-Pad57) -> /IO/DI4
- U2 pad 59: /LTE/LTE_UART_CTS -> /LTE_UART_CTS
- U2 pad 60: unconnected-(U2-PD22-Pad60) -> /IO/DI5
- U2 pad 62: /LTE/LTE_UART_DCD -> /LTE_UART_DCD
- U2 pad 63: unconnected-(U2-PD21-Pad63) -> /IO/DI6
- U2 pad 66: /LTE/LTE_UART_DBG_TXD -> /LTE_UART_DBG_TXD
- U2 pad 67: /RTC_MFP -> unconnected-(U2-PD19-Pad67)
- U2 pad 69: /~{RTD1_DRDY} -> unconnected-(U2-PD18-Pad69)
- U2 pad 70: /LTE/LTE_UART_DTR -> /LTE_UART_DTR
- U2 pad 71: /IO/DI4 -> /IO/DI7
- U2 pad 74: /~{RTD0_DRDY} -> unconnected-(U2-PD17-Pad74)
- U2 pad 75: /LTE/LTE_UART_DBG_RXD -> /LTE_UART_DBG_RXD
- U2 pad 84: /LTE_PWRKEY -> unconnected-(U2-PD14-Pad84)
- U2 pad 88: /LTE_STATUS -> unconnected-(U2-PD13-Pad88)
- U2 pad 92: /LTE_AP_READY -> unconnected-(U2-PD12-Pad92)
- U2 pad 98: /SAM4E_INT -> unconnected-(U2-PD11-Pad98)
- U2 pad 99: /CNT1 -> unconnected-(U2-PA1/PGMEN1-Pad99)
- U5 pad 17: /LTE_STATUS -> /LTE/LTE_STATUS
- U6 pad 6: MCV_CAN0_L -> MCV_CAN1_L
- U6 pad 7: MCV_CAN0_H -> MCV_CAN1_H
- U7 pad 6: MCV_CAN1_L -> MCV_CAN0_L
- U7 pad 7: MCV_CAN1_H -> MCV_CAN0_H
- U8 pad 16: /SPI_CS1 -> /SPI_CS2
Routing:
- net +3V3: track 198.6 -> 572.3 mm, vias 0 -> 5
- net /SPI_MISO: track 0.00 -> 192.7 mm, vias 0 -> 3
- net Net-(U2-VDDIN): track 41.1 -> 231.5 mm, vias 0 -> 7
- net /SPI_SCK: track 0.00 -> 177.3 mm, vias 0 -> 3
- net /SPI_MOSI: track 0.00 -> 174.6 mm, vias 0 -> 3
- net /~{RS_RE}: track 0.00 -> 167.3 mm, vias 0 -> 2
- net /RS_DE: track 0.00 -> 156.1 mm, vias 0 -> 2
- net Net-(U2-VDDOUT): track 48.9 -> 187.7 mm, vias 0 -> 5
- net /ESP32_INT: track 0.00 -> 129.0 mm, vias 0 -> 1
- net /SAM4E_INT: track 0.00 -> 126.1 mm, vias 0 -> 1
- net /~{RTD0_DRDY}: track 0.00 -> 106.0 mm, vias 0 -> 2
- net /CAN0_RS: track 11.8 -> 107.6 mm
- net /CAN0_EN: track 9.88 -> 102.9 mm, vias 1 -> 2
- net /SPI_CS2: track 0.00 -> 89.4 mm, vias 0 -> 2
- net /~{RTD1_DRDY}: track 0.00 -> 88.0 mm, vias 0 -> 2
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
Commit message: [UPDATE]
Work in progress.

Signed-off-by: Nicolae-Andrei Vasile <vasilenicolaeandrei@gmail.com>
Parts:
- removed BT1: CR2032 (Panasonic vertical), Battery:Battery_Panasonic_CR2032-VS1N_Vertical_CircularHoles
- removed C100, C105: 10uF/16V/20%/4x5.4mm, Capacitor_SMD:CP_Elec_4x5.4
- removed C101, C104, C99: 0.1uF/6.3V/20%/C0603, Capacitor_SMD:C_0603_1608Metric
- removed C102, C103: 10pF/6.3V/10%/C0603, Capacitor_SMD:C_0603_1608Metric
- removed the C37 at (-163.6, 106.7)
- removed the C38 at (-163.6, 109.2)
- removed the C39 at (-163.6, 111.7)
- removed the C40 at (-163.6, 114.2)
- removed the C41 at (-163.6, 116.7)
- removed the C42 at (-125.1, 84.2)
- removed the C43 at (-163.6, 119.2)
- removed the C44 at (-163.6, 121.7)
- removed the C45 at (-159.6, 106.7)
- removed the C46 at (-159.6, 109.2)
- removed the C47 at (-159.6, 111.7)
- removed the C48 at (-159.6, 114.2)
- removed the C49 at (-125.1, 90.1)
- removed the C50 at (-159.6, 116.7)
- removed the C51 at (-159.6, 119.2)
- removed the C52 at (-159.6, 121.7)
- removed the C53 at (-155.6, 106.7)
- removed the C54 at (-155.6, 109.2)
- removed the C55 at (-155.6, 111.7)
- removed the C56 at (-155.6, 114.2)
- removed the C57 at (-155.6, 116.7)
- removed the C58 at (-155.6, 119.2)
- removed the C59 at (-155.6, 121.7)
- removed the C60 at (-151.6, 106.7)
- removed C98: 22uF/6.3V/20%/C0603, Capacitor_SMD:C_0603_1608Metric
- removed the D3 at (-126.4, 95.2)
- removed D39: 20V/0.5A/0.5V (NSR0620P2T5G), Diode_SMD:D_SOD-923
- removed the D4 at (-119.3, 114.9)
- removed the J5 at (-137.7, 113.6)
- removed L14, L15: FB0805/600R/2A, Inductor_SMD:L_0805_2012Metric
- removed the L3 at (-118.9, 106.8)
- removed the L4 at (-118.9, 109.5)
- removed the L5 at (-118.9, 112.3)
- removed the Q1 at (-118.8, 83.5)
- removed the Q2 at (-118.8, 88.0)
- removed R115, R116: 10K/R0603, Resistor_SMD:R_0603_1608Metric
- removed the R14 at (-151.6, 109.2)
- removed the R15 at (-151.6, 111.7)
- removed the R16 at (-151.6, 114.2)
- removed the R17 at (-151.6, 116.7)
- removed the R18 at (-151.6, 119.2)
- removed the R19 at (-127.5, 72.3)
- removed the R20 at (-127.5, 74.3)
- removed the R21 at (-127.5, 76.3)
- removed the R22 at (-151.6, 121.7)
- removed the R23 at (-147.6, 106.7)
- removed the R24 at (-147.6, 109.2)
- removed the R25 at (-147.6, 111.7)
- removed the R26 at (-147.6, 114.2)
- removed the R27 at (-127.5, 78.3)
- removed the R28 at (-127.5, 80.3)
- removed the R29 at (-124.6, 72.3)
- removed the R30 at (-124.6, 74.3)
- removed the R31 at (-124.6, 76.3)
- removed the R32 at (-124.6, 78.3)
- removed the R33 at (-124.6, 80.3)
- removed the R34 at (-121.7, 72.3)
- removed the R35 at (-147.6, 116.7)
- removed the R36 at (-147.6, 119.2)
- removed the R37 at (-121.7, 74.3)
- removed the R38 at (-121.7, 76.3)
- removed RV3: V5.5MLA0603N, Resistor_SMD:R_0603_1608Metric
- removed U15: MCP7940N-xSN, Package_SO:SOIC-8_3.9x4.9mm_P1.27mm
- removed U16: 24LC512, Package_SO:SOIC-8_3.9x4.9mm_P1.27mm
- removed the U3 at (-147.3, 88.4)
- removed the U4 at (-125.5, 109.4)
- removed the U5 at (-125.5, 117.5)
- removed XTAL1: ECS-_327-7-34B-TR, digikey-footprints:SMD-2_3.2x1.5mm
- added JP3: SolderJumper_2_Open, Jumper:SolderJumper-2_P1.3mm_Open_Pad1.0x1.5mm, F.Cu at (80.0, 108.0)
- H1, H2, H3, H4: footprint MountingHole:MountingHole_2.5mm -> MountingHole:MountingHole_2.5mm_Pad_Via
- moved R12 2.01 mm to (125.7, 147.3), turned to 90 degrees
- moved D2 1.91 mm to (110.5, 170.2), turned to -90 degrees
- moved R11 1.25 mm to (123.8, 147.3)
- moved C60 0.63 mm to (144.1, 105.4)
- renumbered C61 to C37, C62 to C38, C63 to C39, C64 to C40, C65 to C41, C66 to C42, C67 to C43, C68 to C44, C69 to C45, C70 to C46, C71 to C47, C72 to C48, C73 to C49, C74 to C50, C75 to C51, C76 to C52, C77 to C53, C78 to C54, C79 to C55, C80 to C56, C81 to C57, C82 to C58, C83 to C59, C84 to C60, C85 to C61, C86 to C62, C87 to C63, C88 to C64, C89 to C65, C90 to C66, C91 to C67, C92 to C68, C93 to C69, C94 to C70, C95 to C71, C96 to C72, C97 to C73, D12 to D10, D13 to D11, D14 to D12, D15 to D13, D16 to D14, D17 to D15, D18 to D16, D19 to D17, D20 to D18, D21 to D19, D22 to D20, D23 to D21, D24 to D22, D25 to D23, D26 to D24, D27 to D25, D28 to D26, D29 to D27, D30 to D28, D31 to D29, D5 to D3, D32 to D30, D33 to D31, D34 to D32, D35 to D33, D36 to D34, D37 to D35, D38 to D36, D6 to D4, D7 to D5, D8 to D6, D9 to D7, D10 to D8, D11 to D9, J6 to J5, J7 to J6, J8 to J7, J9 to J8, JP9 to JP10, JP10 to JP11, JP11 to JP12, JP12 to JP13, JP13 to JP14, JP14 to JP15, JP15 to JP16, JP16 to JP17, JP17 to JP18, JP18 to JP19, JP19 to JP20, JP3 to JP4, JP4 to JP5, JP5 to JP6, JP6 to JP7, JP7 to JP8, JP8 to JP9, L13 to L10, L6 to L3, L7 to L4, L8 to L5, L9 to L6, L10 to L7, L11 to L8, L12 to L9, Q3 to Q1, Q12 to Q10, Q13 to Q11, Q4 to Q2, Q5 to Q3, Q6 to Q4, Q7 to Q5, Q8 to Q6, Q9 to Q7, Q10 to Q8, Q11 to Q9, R39 to R14, R40 to R15, R41 to R16, R42 to R17, R43 to R18, R44 to R19, R45 to R20, R46 to R21, R47 to R22, R48 to R23, R49 to R24, R50 to R25, R51 to R26, R52 to R27, R53 to R28, R54 to R29, R55 to R30, R56 to R31, R57 to R32, R58 to R33, R59 to R34, R60 to R35, R61 to R36, R62 to R37, R63 to R38, R64 to R39, R65 to R40, R66 to R41, R67 to R42, R68 to R43, R69 to R44, R70 to R45, R71 to R46, R72 to R47, R73 to R48, R74 to R49, R75 to R50, R76 to R51, R77 to R52, R78 to R53, R79 to R54, R80 to R55, R81 to R56, R82 to R57, R83 to R58, R84 to R59, R85 to R60, R86 to R61, R87 to R62, R88 to R63, R89 to R64, R90 to R65, R91 to R66, R92 to R67, R93 to R68, R94 to R69, R95 to R70, R96 to R71, R97 to R72, R98 to R73, R99 to R74, R100 to R75, R101 to R76, R102 to R77, R103 to R78, R104 to R79, R105 to R80, R106 to R81, R107 to R82, R108 to R83, R109 to R84, R110 to R85, R111 to R86, R112 to R87, R113 to R88, R114 to R89, U13 to U10, U14 to U11, U6 to U3, U7 to U4, U8 to U5, U9 to U6, U10 to U7, U11 to U8, U12 to U9
Connections:
- net /AI0 renamed /IO/AI0
- net /AI1 renamed /IO/AI1
- net /AI2 renamed /IO/AI2
- net /AI3 renamed /IO/AI3
- J3 pad 10: GND -> /SPI_MOSI
- J3 pad 3: unconnected-(J3-Pin_3-Pad3) -> /SAM4E_INT
- J3 pad 4: /ESP32_INT -> /SPI_CS0
- J3 pad 5: unconnected-(J3-Pin_5-Pad5) -> /ESP32_INT
- J3 pad 6: /SAM4E_INT -> /SPI_MISO
- J3 pad 7: unconnected-(J3-Pin_7-Pad7) -> GND
- J3 pad 8: GND -> /SPI_SCK
- J3 pad 9: unconnected-(J3-Pin_9-Pad9) -> GND
- J4 pad 10: unconnected-(J4-Pin_10-Pad10) -> /LTE_UART_TXD
- J4 pad 12: unconnected-(J4-Pin_12-Pad12) -> /LTE_UART_RXD
- J4 pad 6: unconnected-(J4-Pin_6-Pad6) -> /LTE_UART_RI
- J4 pad 8: unconnected-(J4-Pin_8-Pad8) -> /LTE_UART_RTS
- J5 pad 5: /IO/MCV_DO1 -> /IO/MCV_DO2
- J5 pad 6: /IO/MCV_DO2 -> /IO/MCV_DO1
Routing:
- net /LTE_UART_RI: track 34.1 -> 220.1 mm, vias 1 -> 2
- net +3V3: track 572.3 -> 610.4 mm
- net /LTE_UART_TXD: track 41.8 -> 71.2 mm
- net /SPI_MOSI: track 174.6 -> 203.0 mm
- net /LTE_UART_RXD: track 43.9 -> 71.7 mm
- net /SPI_SCK: track 177.3 -> 203.5 mm
- net /LTE_UART_RTS: track 68.9 -> 91.1 mm
- net /SPI_MISO: track 192.7 -> 213.4 mm
- net /CAN0_D: track 66.0 -> 83.0 mm
- net /CAN0_R: track 58.4 -> 74.1 mm
- net /SPI_CS0: track 79.8 -> 93.7 mm
- net /I2C_SDA: track 75.4 -> 88.9 mm, vias 1 -> 2
- net Net-(D2-K): track 0.00 -> 13.0 mm
- net /I2C_SCL: track 87.2 -> 100.1 mm, vias 1 -> 2
- net Net-(D1-K): track 0.00 -> 10.0 mm
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