File: board-design/kicad-files/SAM4E-PLC/IO.kicad_sch (KiCad schematic)
At the start: 126 parts, among them Q1 BC807, Q10 BC807, Q2 BC807, Q3 BC807, Q4 BC807, Q5 BC807, Q6 BC807, Q7 BC807, Q8 BC807, Q9 BC807, U10 SN74HC240DBR, U8 ULN2803CDWR, U9 74AC14SCX

Commit message: [UPDATE]
Completed SAM4E-PLC board design.

Signed-off-by: Nicolae-Andrei Vasile <vasilenicolaeandrei@gmail.com>
Other:
- title: (none) -> SAM4E

Commit message: [Final report]
Added 3D models.

Signed-off-by: Nicolae-Andrei Vasile <vasilenicolaeandrei@gmail.com>
Parts:
- gave numbers to parts that had none: 6
- renumbered C4 to C58, C37 to C59, C38 to C60, C37 to C61, C38 to C62, C5 to C63, C5 to C64, C5 to C65, C5 to C66, R9 to R54, R9 to R55, R9 to R56, R9 to R57, R9 to R58, R9 to R59, R9 to R60, R9 to R61, R9 to R62, R9 to R63, R9 to R64, R9 to R65, R9 to R66, R9 to R67, R9 to R68, R9 to R69, R9 to R74, R9 to R75, R9 to R76, R9 to R77
