File: board-design/kicad-files/SAM4E-PLC/PWR.kicad_sch (KiCad schematic)
At the start: 18 parts, among them Q11 BC817, U11 LM2576HVS-3.3

Commit message: [Final report]
Added 3D models.

Signed-off-by: Nicolae-Andrei Vasile <vasilenicolaeandrei@gmail.com>
Parts:
- renumbered C5 to C67, C5 to C68, C5 to C69, C5 to C70, C5 to C71, C37 to C72, C37 to C73, D35 to D36, F9 to F13, R48 to R86, R9 to R87, R9 to R88
Changed lines of the file:
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@@
   (symbol (lib_id "Device:C_Polarized") (at 196.85 104.14 0) (unit 1)
     (in_bom yes) (on_board yes) (dnp no)
-    (property "Reference" "C5" (at 198.12 109.22 90)
+    (property "Reference" "C71" (at 198.12 109.22 90)
       (effects (font (size 1.27 1.27)) (justify left))
     )
@@
     (instances
       (project "SAM4E-PLC"
-        (path "/93076d8a-73da-4f5d-b7f2-28678f1db77d/32910dfe-b730-4651-8391-975b8cdac59d"
-          (reference "C5") (unit 1)
-        )
         (path "/93076d8a-73da-4f5d-b7f2-28678f1db77d/aee81a7b-cba1-4b89-a883-459d3f783e91"
           (reference "C71") (unit 1)
@@
   (symbol (lib_id "Device:C_Polarized") (at 95.25 99.06 0) (unit 1)
     (in_bom yes) (on_board yes) (dnp no)
-    (property "Reference" "C5" (at 96.52 104.14 90)
+    (property "Reference" "C68" (at 96.52 104.14 90)
       (effects (font (size 1.27 1.27)) (justify left))
     )
@@
     (instances
       (project "SAM4E-PLC"
-        (path "/93076d8a-73da-4f5d-b7f2-28678f1db77d/32910dfe-b730-4651-8391-975b8cdac59d"
-          (reference "C5") (unit 1)
-        )
         (path "/93076d8a-73da-4f5d-b7f2-28678f1db77d/aee81a7b-cba1-4b89-a883-459d3f783e91"
           (reference "C68") (unit 1)
@@
   (symbol (lib_id "Device:C") (at 209.55 104.14 0) (unit 1)
     (in_bom yes) (on_board yes) (dnp no)
-    (property "Reference" "C37" (at 210.82 109.22 90)
+    (property "Reference" "C73" (at 210.82 109.22 90)
       (effects (font (size 1.27 1.27)) (justify left))
     )
@@
     (instances
       (project "SAM4E-PLC"
-        (path "/93076d8a-73da-4f5d-b7f2-28678f1db77d/32910dfe-b730-4651-8391-975b8cdac59d"
-          (reference "C37") (unit 1)
-        )
-        (path "/93076d8a-73da-4f5d-b7f2-28678f1db77d/f76e13f7-6a24-4ea6-98c5-a4d0bd3b3ced"
-          (reference "C55") (unit 1)
-        )
         (path "/93076d8a-73da-4f5d-b7f2-28678f1db77d/aee81a7b-cba1-4b89-a883-459d3f783e91"
           (reference "C73") (unit 1)
@@
   (symbol (lib_id "Device:C_Polarized") (at 165.1 104.14 0) (unit 1)
     (in_bom yes) (on_board yes) (dnp no)
-    (property "Reference" "C5" (at 166.37 109.22 90)
+    (property "Reference" "C69" (at 166.37 109.22 90)
       (effects (font (size 1.27 1.27)) (justify left))
     )
@@
     (instances
       (project "SAM4E-PLC"
-        (path "/93076d8a-73da-4f5d-b7f2-28678f1db77d/32910dfe-b730-4651-8391-975b8cdac59d"
-          (reference "C5") (unit 1)
-        )
         (path "/93076d8a-73da-4f5d-b7f2-28678f1db77d/aee81a7b-cba1-4b89-a883-459d3f783e91"
           (reference "C69") (unit 1)
@@
   (symbol (lib_id "Device:Fuse") (at 44.45 92.71 90) (unit 1)
     (in_bom yes) (on_board yes) (dnp no)
-    (property "Reference" "F9" (at 44.45 87.63 90)
+    (property "Reference" "F13" (at 44.45 87.63 90)
       (effects (font (size 1.27 1.27)))
     )
@@
     (instances
       (project "SAM4E-PLC"
-        (path "/93076d8a-73da-4f5d-b7f2-28678f1db77d/f76e13f7-6a24-4ea6-98c5-a4d0bd3b3ced"
-          (reference "F9") (unit 1)
-        )
         (path "/93076d8a-73da-4f5d-b7f2-28678f1db77d/aee81a7b-cba1-4b89-a883-459d3f783e91"
           (reference "F13") (unit 1)
@@
   (symbol (lib_id "Device:C_Polarized") (at 88.9 99.06 0) (unit 1)
     (in_bom yes) (on_board yes) (dnp no)
-    (property "Reference" "C5" (at 90.17 104.14 90)
+    (property "Reference" "C67" (at 90.17 104.14 90)
       (effects (font (size 1.27 1.27)) (justify left))
     )
@@
     (instances
       (project "SAM4E-PLC"
-        (path "/93076d8a-73da-4f5d-b7f2-28678f1db77d/32910dfe-b730-4651-8391-975b8cdac59d"
-          (reference "C5") (unit 1)
-        )
         (path "/93076d8a-73da-4f5d-b7f2-28678f1db77d/aee81a7b-cba1-4b89-a883-459d3f783e91"
           (reference "C67") (unit 1)
@@
   (symbol (lib_id "Device:R") (at 234.95 104.14 0) (unit 1)
     (in_bom yes) (on_board yes) (dnp no)
-    (property "Reference" "R9" (at 232.41 102.87 0)
+    (property "Reference" "R87" (at 232.41 102.87 0)
       (effects (font (size 1.27 1.27)) (justify right))
     )
@@
     (instances
       (project "SAM4E-PLC"
-        (path "/93076d8a-73da-4f5d-b7f2-28678f1db77d/32910dfe-b730-4651-8391-975b8cdac59d"
-          (reference "R9") (unit 1)
-        )
-        (path "/93076d8a-73da-4f5d-b7f2-28678f1db77d/f76e13f7-6a24-4ea6-98c5-a4d0bd3b3ced"
-          (reference "R88") (unit 1)
-        )
         (path "/93076d8a-73da-4f5d-b7f2-28678f1db77d/aee81a7b-cba1-4b89-a883-459d3f783e91"
           (reference "R87") (unit 1)
@@
   (symbol (lib_id "Device:R") (at 245.11 104.14 0) (unit 1)
     (in_bom yes) (on_board yes) (dnp no)
-    (property "Reference" "R9" (at 247.015 102.87 0)
+    (property "Reference" "R88" (at 247.015 102.87 0)
       (effects (font (size 1.27 1.27)) (justify left))
     )
@@
     (instances
       (project "SAM4E-PLC"
-        (path "/93076d8a-73da-4f5d-b7f2-28678f1db77d/32910dfe-b730-4651-8391-975b8cdac59d"
-          (reference "R9") (unit 1)
-        )
-        (path "/93076d8a-73da-4f5d-b7f2-28678f1db77d/f76e13f7-6a24-4ea6-98c5-a4d0bd3b3ced"
-          (reference "R88") (unit 1)
-        )
         (path "/93076d8a-73da-4f5d-b7f2-28678f1db77d/aee81a7b-cba1-4b89-a883-459d3f783e91"
           (reference "R88") (unit 1)
@@
       )
       (project "SAM4E-PLC"
-        (path "/93076d8a-73da-4f5d-b7f2-28678f1db77d/f76e13f7-6a24-4ea6-98c5-a4d0bd3b3ced"
-          (reference "R53") (unit 1)
-        )
         (path "/93076d8a-73da-4f5d-b7f2-28678f1db77d/aee81a7b-cba1-4b89-a883-459d3f783e91"
           (reference "R89") (unit 1)
@@
   (symbol (lib_id "Device:C") (at 203.2 104.14 0) (unit 1)
     (in_bom yes) (on_board yes) (dnp no)
-    (property "Reference" "C37" (at 204.47 109.22 90)
+    (property "Reference" "C72" (at 204.47 109.22 90)
       (effects (font (size 1.27 1.27)) (justify left))
     )
@@
     (instances
       (project "SAM4E-PLC"
-        (path "/93076d8a-73da-4f5d-b7f2-28678f1db77d/32910dfe-b730-4651-8391-975b8cdac59d"
-          (reference "C37") (unit 1)
-        )
-        (path "/93076d8a-73da-4f5d-b7f2-28678f1db77d/f76e13f7-6a24-4ea6-98c5-a4d0bd3b3ced"
-          (reference "C55") (unit 1)
-        )
         (path "/93076d8a-73da-4f5d-b7f2-28678f1db77d/aee81a7b-cba1-4b89-a883-459d3f783e91"
           (reference "C72") (unit 1)
@@
   (symbol (lib_id "Device:C_Polarized") (at 171.45 104.14 0) (unit 1)
     (in_bom yes) (on_board yes) (dnp no)
-    (property "Reference" "C5" (at 172.72 109.22 90)
+    (property "Reference" "C70" (at 172.72 109.22 90)
       (effects (font (size 1.27 1.27)) (justify left))
     )
@@
     (instances
       (project "SAM4E-PLC"
-        (path "/93076d8a-73da-4f5d-b7f2-28678f1db77d/32910dfe-b730-4651-8391-975b8cdac59d"
-          (reference "C5") (unit 1)
-        )
         (path "/93076d8a-73da-4f5d-b7f2-28678f1db77d/aee81a7b-cba1-4b89-a883-459d3f783e91"
           (reference "C70") (unit 1)
@@
   (symbol (lib_id "Device:LED") (at 234.95 114.3 90) (unit 1)
     (in_bom yes) (on_board yes) (dnp no)
-    (property "Reference" "D35" (at 232.41 113.03 90)
+    (property "Reference" "D36" (at 232.41 113.03 90)
       (effects (font (size 1.27 1.27)) (justify left))
     )
@@
     (instances
       (project "SAM4E-PLC"
-        (path "/93076d8a-73da-4f5d-b7f2-28678f1db77d/f76e13f7-6a24-4ea6-98c5-a4d0bd3b3ced"
-          (reference "D35") (unit 1)
-        )
         (path "/93076d8a-73da-4f5d-b7f2-28678f1db77d/aee81a7b-cba1-4b89-a883-459d3f783e91"
           (reference "D36") (unit 1)
@@
   (symbol (lib_id "Device:R") (at 184.15 97.79 90) (mirror x) (unit 1)
     (in_bom yes) (on_board yes) (dnp no)
-    (property "Reference" "R48" (at 185.42 95.25 90)
+    (property "Reference" "R86" (at 185.42 95.25 90)
       (effects (font (size 1.27 1.27)) (justify left))
     )
@@
     (instances
       (project "SAM4E-PLC"
-        (path "/93076d8a-73da-4f5d-b7f2-28678f1db77d/32910dfe-b730-4651-8391-975b8cdac59d"
-          (reference "R48") (unit 1)
-        )
         (path "/93076d8a-73da-4f5d-b7f2-28678f1db77d/aee81a7b-cba1-4b89-a883-459d3f783e91"
           (reference "R86") (unit 1)
@@
   (symbol (lib_id "power:PWR_FLAG") (at 111.76 90.17 0) (unit 1)
     (in_bom yes) (on_board yes) (dnp no) (fields_autoplaced)
-    (property "Reference" "#FLG016" (at 111.76 88.265 0)
+    (property "Reference" "#FLG013" (at 111.76 88.265 0)
       (effects (font (size 1.27 1.27)) hide)
     )
@@
     (instances
       (project "SAM4E-PLC"
-        (path "/93076d8a-73da-4f5d-b7f2-28678f1db77d/f76e13f7-6a24-4ea6-98c5-a4d0bd3b3ced"
-          (reference "#FLG016") (unit 1)
-        )
         (path "/93076d8a-73da-4f5d-b7f2-28678f1db77d/aee81a7b-cba1-4b89-a883-459d3f783e91"
           (reference "#FLG013") (unit 1)
